Commit message: feat: replace primitive box with real VN-100 Rugged 3D mesh
Convert vn100_rugged.step to STL via gmsh (scale 0.001 mm→m).
Update URDF to reference the mesh so Foxglove and RViz render
the actual sensor geometry rotating with the dynamic TF.

File: ros2_ws/src/imu_dds_adapter/urdf/vn100.urdf (robot description, URDF)
Before this commit: robot vn100_imu, 1 links, 0 joints
Links:
- link imu_link: geometry visual mesh filename=package://imu_dds_adapter/meshes/vn100_rugged.stl scale=0.001 0.001 0.001
